File: case_elec/odb.kicad_sch (KiCad schematic)
At the start: 9 parts, among them J1 Screw_Terminal_01x02, J2 Conn_02x07_Top_Bottom, SW1 SW_SPST, SW2 SW_SPST, U1 REYAX RYLR896, U2 BNO055, U3 MPL3115A, U4 Ultimate_GPS, U5 Teensy3.5

Commit message: pcb en cours de tracé
Connections:
- net at U3.8 (SCL), U5.9 (7_RX3_MOSI0_SCL0): now also U2.5 (SCL); no longer U2.4 (SCL)
- net at U3.7 (SDA), U5.10 (8_TX3_MISO0_SDA0): now also U2.4 (SDA); no longer U2.5 (SDA)
Changed lines of the file:
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@@
   (junction (at 78.74 81.28) (diameter 0) (color 0 0 0 0)
   )
+  (junction (at 107.95 63.5) (diameter 0) (color 0 0 0 0)
+  )
+  (junction (at 144.78 153.67) (diameter 0) (color 0 0 0 0)
+  )
   (junction (at 110.49 60.96) (diameter 0) (color 0 0 0 0)
   )
-  (junction (at 144.78 153.67) (diameter 0) (color 0 0 0 0)
-  )
-  (junction (at 107.95 63.5) (diameter 0) (color 0 0 0 0)
-  )
   (bus_entry (at 167.64 158.75) (size 2.54 -2.54)
     (stroke (width 0) (type default) (color 0 0 0 0))
@@
     (stroke (width 0) (type default) (color 0 0 0 0))
   )
-  (wire (pts (xy 110.49 83.82) (xy 110.49 60.96))
+  (wire (pts (xy 107.95 83.82) (xy 107.95 63.5))
     (stroke (width 0) (type default) (color 0 0 0 0))
   )
@@
     (stroke (width 0) (type default) (color 0 0 0 0))
   )
+  (wire (pts (xy 110.49 60.96) (xy 110.49 86.36))
+    (stroke (width 0) (type default) (color 0 0 0 0))
+  )
   (wire (pts (xy 209.55 130.81) (xy 213.36 130.81))
     (stroke (width 0) (type default) (color 0 0 0 0))
@@
     (stroke (width 0) (type default) (color 0 0 0 0))
   )
-  (wire (pts (xy 110.49 83.82) (xy 99.06 83.82))
+  (wire (pts (xy 107.95 83.82) (xy 99.06 83.82))
     (stroke (width 0) (type default) (color 0 0 0 0))
   )
@@
     (stroke (width 0) (type default) (color 0 0 0 0))
   )
-  (wire (pts (xy 107.95 86.36) (xy 99.06 86.36))
+  (wire (pts (xy 99.06 86.36) (xy 110.49 86.36))
     (stroke (width 0) (type default) (color 0 0 0 0))
   )
@@
     (stroke (width 0) (type default) (color 0 0 0 0))
   )
-  (wire (pts (xy 107.95 86.36) (xy 107.95 63.5))
-    (stroke (width 0) (type default) (color 0 0 0 0))
-  )
   (wire (pts (xy 209.55 140.97) (xy 213.36 140.97))
     (stroke (width 0) (type default) (color 0 0 0 0))
@@
     (stroke (width 0) (type default) (color 0 0 0 0))
   )
+  (wire (pts (xy 107.95 54.61) (xy 107.95 63.5))
+    (stroke (width 0) (type default) (color 0 0 0 0))
+  )
   (bus (pts (xy 144.78 138.43) (xy 144.78 140.97))
     (stroke (width 0) (type default) (color 0 0 0 0))
   )
+  (wire (pts (xy 97.79 60.96) (xy 110.49 60.96))
+    (stroke (width 0) (type default) (color 0 0 0 0))
+  )
   (wire (pts (xy 110.49 57.15) (xy 110.49 60.96))
     (stroke (width 0) (type default) (color 0 0 0 0))
@@
   )
   (wire (pts (xy 134.62 90.17) (xy 151.13 90.17))
-    (stroke (width 0) (type default) (color 0 0 0 0))
-  )
-  (wire (pts (xy 110.49 60.96) (xy 97.79 60.96))
-    (stroke (width 0) (type default) (color 0 0 0 0))
-  )
-  (wire (pts (xy 107.95 54.61) (xy 107.95 63.5))
     (stroke (width 0) (type default) (color 0 0 0 0))
   )
@@
     (pin "9")
   )
-  (symbol (lib_name "BNO055_1") (lib_id "Adafruit_sensors:BNO055") (at 88.9 88.9 180) (unit 1)
+  (symbol (lib_id "Adafruit_sensors:BNO055") (at 88.9 88.9 180) (unit 1)
     (in_bom yes) (on_board yes)
     (property "Reference" "U2" (id 0) (at 88.9 99.06 0))
@@
       (effects (font (size 1.27 1.27)) hide)
     )
-    (property "Datasheet" "https://cdn-learn.adafruit.com/assets/assets/000/036/832/original/BST_BNO055_DS000_14.pdf" (id 3) (at 80.01 102.87 0))
+    (property "Datasheet" "https://cdn-learn.adafruit.com/downloads/pdf/adafruit-bno055-absolute-orientation-sensor.pdf" (id 3) (at 80.01 102.87 0))
     (pin "1")
     (pin "10")

Commit message: complétion du pcb
Connections:
- net +5V: now also U4.8 (VIN); no longer U4.7 (VIN)
- net GND: now also U4.7 (GND); no longer U4.6 (GND)
- net at U5.2 (0_RX1_MOSI1_Touch): now also U4.5 (TX); no longer U4.4 (TX)
- net at U5.3 (1_TX1_MISO1_Touch): now also U4.6 (RX); no longer U4.5 (RX)
Changed lines of the file:
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@@
     (pin "3")
-    (pin "4")
     (pin "4")
     (pin "5")
@@
     (pin "7")
     (pin "8")
+    (pin "9")
   )
   (symbol (lib_id "Switch:SW_SPST") (at 64.77 81.28 0) (mirror x) (unit 1)
