File: case_elec/seq/seq.kicad_sch (KiCad schematic)
At the start: 15 parts, among them J1 LiPo, J10 Coupleur, J11 Jack, J2 B-, J3 BM, J4 B+, J5 P+, J6 P-, J7 Servo, J8 LEDs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

Commit message: sauvetage, màj seq version à usiner
Parts:
- added J2: Lipo Alim, Connector_PinHeader_2.54mm:PinHeader_1x03_P2.54mm_Vertical, symbol Connector:Conn_01x03_Male
- J1: value LiPo -> LiPo BMS; footprint Connector_JST:JST_EH_B3B-EH-A_1x03_P2.50mm_Vertical -> Connector_JST:JST_XH_B3B-XH-A_1x03_P2.50mm_Vertical
- J10: renamed from J9; footprint TerminalBlock_Phoenix:TerminalBlock_Phoenix_MKDS-1,5-2-5.08_1x02_P5.08mm_Horizontal -> Connector_PinHeader_2.54mm:PinHeader_1x03_P2.54mm_Vertical; symbol Connector:Screw_Terminal_01x02 -> Connector:Conn_01x03_Male
- J12: renamed from J11; footprint Connector_JST:JST_EH_B3B-EH-A_1x03_P2.50mm_Vertical -> Connector_JST:JST_XH_B2B-XH-A_1x02_P2.50mm_Vertical; symbol Connector:Conn_01x03_Male -> Connector:Conn_01x02_Male
- J8: renamed from J7; footprint Connector_JST:JST_EH_B3B-EH-A_1x03_P2.50mm_Vertical -> Connector_JST:JST_XH_B3B-XH-A_1x03_P2.50mm_Vertical
- J9: renamed from J8; footprint Connector_JST:JST_EH_B4B-EH-A_1x04_P2.50mm_Vertical -> Connector_JST:JST_XH_B4B-XH-A_1x04_P2.50mm_Vertical
- renumbered J10 to J11, J4 to J3, J3 to J4, J2 to J5, J5 to J6, J6 to J7
Connections:
- net B+: now reaches J3.1 (Pin_1)
- net B+: now also J1.1 (Pin_1), J2.2 (Pin_2); no longer J1.3 (Pin_3)
- net B-: now reaches J5.1 (Pin_1)
- net B-: now also J1.3 (Pin_3), J2.1 (Pin_1); no longer J1.1 (Pin_1)
- net BM: now reaches J1.2 (Pin_2), J4.1 (Pin_1)
Other:
- note removed: "Sorties BMS cas nominal : broches cas échéant : bornier"
- moved on the sheet: J1, J3, J4, J5, J6, J7
