File: case_elec/odb/odb.kicad_pcb (KiCad board)
At the start: 2 copper layers, 98 x 79 mm, 10 parts, among them J1 Screw_Terminal_01x02, J2 Conn_02x07_Top_Bottom, SW1 SW_SPST, SW2 SW_SPST, U1 REYAX RYLR896, U2 BNO055, U3 MPL3115A, U4 Ultimate_GPS, U5 Teensy3.5

Commit message: Ajout d'une piste SCL pour l'alitmètre en panique
Connections:
- U3 pad 6: unconnected-(U3-Pad6) -> Net-(U2-Pad5)
- U5 pad 3: unconnected-(U4-Pad6) -> unconnected-(U5-Pad3)
Routing:
- net Net-(U2-Pad5): track 44.3 -> 66.5 mm
- net unconnected-(U5-Pad3): track 0.00 -> 9.36 mm
- net unconnected-(U4-Pad6): track 9.36 -> 0.00 mm
